File: EL87/EL87.sch (KiCad schematic (older format))
At the start: 201 parts

Commit message: Preliminary PCB layout
Connections:
- net R2: now also D21.1 (K), D22.1 (K), D33.1 (K), D34.1 (K), D35.1 (K)
- net R3: now also D40.1 (K)
- net R6: now also D98.1 (K)
Changed lines of the file:
@@
 Connection ~ 18700 1900
 Wire Wire Line
-	1300 3400 15500 3400
-Wire Wire Line
-	17700 3400 19700 3400
+	1300 3400 19700 3400
 Connection ~ 3500 3400
 Connection ~ 4500 3400
@@
 C17
 Connection ~ 2700 3100
+Connection ~ 6500 3400
+Connection ~ 7500 3400
+Connection ~ 7000 4400
+Connection ~ 16300 7400
 $EndSCHEMATC
