File: EL87/controller.sch (KiCad schematic (older format))
At the start: 165 parts, among them P1 USB_OTG, P2 CONN_02X03, P3 CONN_02X05, P4 CONN_01X03, SW1 SW_PUSH, U1 AT90USB1286, U2 IS31FL3731, U3 IS31FL3731, Y1 16Mhz

Commit message: Preliminary PCB layout
Parts:
- added P5: CONN_01X05, Connectors_Molex:Molex_PicoBlade_53261-0571_05x1.25mm_Angled, symbol CONN_01X05
Connections:
- net GND: now also P5.5 (P5)
- net USB+: now also P1.3 (D+), P5.3 (P3); no longer P1.4 (ID)
- net USB-: now also P1.2 (D-), P5.2 (P2); no longer P1.3 (D+)
- net VBUS: now reaches F1.1, P1.1 (VBUS)
- net VBUS: now also P5.1 (P1)
- new net ID: P1.4 (ID), P5.4 (P4)
Other:
- moved on the sheet: F1, R4, R5
Changed lines of the file:
@@
 L R R4
 U 1 1 581B462B
+P 19400 12100
+F 0 "R4" V 19350 11950 50  0000 C CNN
+F 1 "22Ω" V 19400 12100 50  0000 C CNN
+F 2 "Resistors_SMD:R_0805_HandSoldering" V 19330 12100 50  0001 C CNN
+F 3 "" H 19400 12100 50  0000 C CNN
+	1    19400 12100
+	0    1    1    0
+$EndComp
+$Comp
+L R R5
+U 1 1 581B462C
 P 19400 12200
-F 0 "R4" V 19350 12050 50  0000 C CNN
+F 0 "R5" V 19450 12050 50  0000 C CNN
 F 1 "22Ω" V 19400 12200 50  0000 C CNN
 F 2 "Resistors_SMD:R_0805_HandSoldering" V 19330 12200 50  0001 C CNN
 F 3 "" H 19400 12200 50  0000 C CNN
 	1    19400 12200
-	0    1    1    0
-$EndComp
-$Comp
-L R R5
-U 1 1 581B462C
-P 19400 12300
-F 0 "R5" V 19450 12150 50  0000 C CNN
-F 1 "22Ω" V 19400 12300 50  0000 C CNN
-F 2 "Resistors_SMD:R_0805_HandSoldering" V 19330 12300 50  0001 C CNN
-F 3 "" H 19400 12300 50  0000 C CNN
-	1    19400 12300
 	0    1    1    0
 $EndComp
@@
 	1    0    0    -1
 $EndComp
-Text GLabel 18950 12400 3    60   Input ~ 0
+Text GLabel 18950 12300 3    60   Input ~ 0
 USB+
-Text GLabel 19100 12400 3    60   Input ~ 0
+Text GLabel 19100 12300 3    60   Input ~ 0
 USB-
+Text GLabel 19550 12100 2    60   Input ~ 0
+D-
 Text GLabel 19550 12200 2    60   Input ~ 0
-D-
-Text GLabel 19550 12300 2    60   Input ~ 0
 D+
 $Comp
 L FP_Small F1
 U 1 1 581B462E
-P 18800 12000
-F 0 "F1" H 18760 12060 50  0000 L CNN
-F 1 "FP_Small" H 18680 11940 50  0000 L CNN
-F 2 "Resistors_SMD:R_1206_HandSoldering" H 18800 12000 50  0001 C CNN
-F 3 "" H 18800 12000 50  0000 C CNN
-	1    18800 12000
+P 19000 12000
+F 0 "F1" H 18960 12060 50  0000 L CNN
+F 1 "FP_Small" H 18880 11940 50  0000 L CNN
+F 2 "Resistors_SMD:R_1206_HandSoldering" H 19000 12000 50  0001 C CNN
+F 3 "" H 19000 12000 50  0000 C CNN
+	1    19000 12000
 	1    0    0    -1
 $EndComp
@@
 L +5V #PWR017
 U 1 1 581B462F
-P 18950 11850
-F 0 "#PWR017" H 18950 11700 50  0001 C CNN
-F 1 "+5V" H 18950 11990 50  0000 C CNN
-F 2 "" H 18950 11850 50  0000 C CNN
-F 3 "" H 18950 11850 50  0000 C CNN
-	1    18950 11850
+P 19150 11850
+F 0 "#PWR017" H 19150 11700 50  0001 C CNN
+F 1 "+5V" H 19150 11990 50  0000 C CNN
+F 2 "" H 19150 11850 50  0000 C CNN
+F 3 "" H 19150 11850 50  0000 C CNN
+	1    19150 11850
 	1    0    0    -1
 $EndComp
@@
 Connection ~ 18800 12600
 Wire Wire Line
-	18700 12300 19250 12300
-Wire Wire Line
-	18950 12300 18950 12400
-Wire Wire Line
 	18700 12200 19250 12200
 Wire Wire Line
-	19100 12200 19100 12400
-Connection ~ 18950 12300
-Connection ~ 19100 12200
-Wire Wire Line
-	18900 12000 18950 12000
-Wire Wire Line
-	18950 12000 18950 11850
+	18950 12200 18950 12300
+Wire Wire Line
+	18700 12100 19250 12100
+Wire Wire Line
+	19100 12100 19100 12300
+Connection ~ 18950 12200
+Connection ~ 19100 12100
+Wire Wire Line
+	19100 12000 19150 12000
+Wire Wire Line
+	19150 12000 19150 11850
 Wire Wire Line
 	20800 12300 20800 12200
@@
 Wire Wire Line
 	18700 12400 18800 12400
+$Comp
+L CONN_01X05 P5
+U 1 1 588C123F
+P 15600 11800
+F 0 "P5" H 15600 12100 50  0000 C CNN
+F 1 "CONN_01X05" V 15700 11800 50  0000 C CNN
+F 2 "Connectors_Molex:Molex_PicoBlade_53261-0571_05x1.25mm_Angled" H 15600 11800 50  0001 C CNN
+F 3 "" H 15600 11800 50  0000 C CNN
+	1    15600 11800
+	-1   0    0    -1
+$EndComp
+Text GLabel 15800 11600 2    60   Input ~ 0
+VBUS
+Text GLabel 15800 11700 2    60   Input ~ 0
+USB-
+Text GLabel 15800 11800 2    60   Input ~ 0
+USB+
+$Comp
+L GND #PWR028
+U 1 1 588C1D07
+P 15900 12100
+F 0 "#PWR028" H 15900 11850 50  0001 C CNN
+F 1 "GND" H 15900 11950 50  0000 C CNN
+F 2 "" H 15900 12100 50  0000 C CNN
+F 3 "" H 15900 12100 50  0000 C CNN
+	1    15900 12100
+	1    0    0    -1
+$EndComp
+Wire Wire Line
+	15800 12000 15900 12000
+Wire Wire Line
+	15900 12000 15900 12100
+Text GLabel 18800 11900 1    60   Input ~ 0
+VBUS
+Wire Wire Line
+	18700 12000 18900 12000
+Wire Wire Line
+	18800 12000 18800 11900
+Connection ~ 18800 12000
+Text GLabel 15800 11900 2    60   Input ~ 0
+ID
+Text GLabel 18700 12300 2    60   Input ~ 0
+ID
 $EndSCHEMATC
