File: EL87/EL87.kicad_pcb (KiCad board)
At the start: 2 copper layers, 272 parts, among them P1 USB_OTG, P2 CONN_02X03, P3 CONN_02X05, P4 CONN_01X03, SW1 SW_PUSH, U1 AT90USB1286, U2 IS31FL3731, U3 IS31FL3731, Y1 16Mhz

Commit message: Preliminary PCB layout
Parts:
- removed D30, D68, D73, D86: D, Diodes_SMD:MiniMELF_Standard
- added P5: CONN_01X05, Connectors_Molex:Molex_PicoBlade_53261-0571_05x1.25mm_Angled, B.Cu at (147.6, 32.3)
- C1, C2, C3, C4, C5, C6, C7, C8, C9, F1, P1, P2, P3, R4, R5, U1, Y1: moved to B.Cu
- D55: moved to F.Cu
- moved C11 477.7 mm to (475.1, 49.7)
- moved R8 477.2 mm to (475.2, 43.3)
- moved R6 477.1 mm to (475.7, 37.0)
- moved R3 476.7 mm to (475.7, 30.6)
- moved RGB6 470.0 mm to (467.9, 44.4)
- moved RGB4 469.6 mm to (468.4, 34.0)
- moved R13 469.6 mm to (465.8, 59.8)
- moved RGB10 469.0 mm to (468.4, 23.6)
- moved R7 468.8 mm to (465.8, 53.4)
- moved C15 466.3 mm to (461.6, 66.1)
- moved RGB5 461.7 mm to (458.5, 54.8)
- moved C10 461.6 mm to (456.2, 70.2)
- moved R12 460.7 mm to (456.3, 63.8)
- moved RGB17 460.6 mm to (458.5, 44.4)
- moved RGB9 460.2 mm to (458.9, 34.0)
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Connections:
- net Net-(F1-Pad1) renamed VBUS
- D21 pad 1: Net-(D21-Pad1) -> R2
- D22 pad 1: Net-(D22-Pad1) -> R2
- D33 pad 1: Net-(D33-Pad1) -> R2
- D34 pad 1: Net-(D33-Pad1) -> R2
- D35 pad 1: Net-(D33-Pad1) -> R2
- D40 pad 1: Net-(D40-Pad1) -> R3
- D98 pad 1: Net-(D98-Pad1) -> R6
- P1 pad 2: Net-(P1-Pad2) -> USB-
- P1 pad 3: USB- -> USB+
- P1 pad 4: USB+ -> ID
- P2 pad : (no net) -> GND
Routing:
- net R5: track 0.00 -> 409.5 mm, vias 0 -> 2
- net R4: track 0.00 -> 374.8 mm, vias 0 -> 2
- net R6: track 0.00 -> 358.4 mm, vias 0 -> 2
- net R2: track 0.00 -> 351.7 mm, vias 0 -> 2
- net R3: track 0.00 -> 341.8 mm, vias 0 -> 2
- net C1: track 0.00 -> 307.3 mm, vias 0 -> 1
- net C2: track 0.00 -> 265.9 mm, vias 0 -> 1
- net C3: track 0.00 -> 265.5 mm, vias 0 -> 1
- net R1: track 0.00 -> 252.4 mm
- net C17: track 0.00 -> 239.8 mm, vias 0 -> 1
- net C4: track 0.00 -> 225.1 mm, vias 0 -> 1
- net C16: track 0.00 -> 219.7 mm, vias 0 -> 1
- net C5: track 0.00 -> 207.6 mm, vias 0 -> 1
- net C15: track 0.00 -> 199.8 mm, vias 0 -> 1
- net C7: track 0.00 -> 195.4 mm, vias 0 -> 1
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- added copper zone on B.Cu, net GND
- added copper zone on F.Cu, net GND
Other:
- board outline added: 347.3 x 123.6 mm
- net class 10m: via_dia 0.6096 -> 0.6858; via_drill 0.3048 -> 0.3302
- net class 20m: clearance 0.254 -> 0.2032; via_dia 0.6096 -> 0.6858; via_drill 0.3048 -> 0.3302
- net class 8mm added: clearance 0.2032, trace_width 0.2032, via_dia 0.6858, via_drill 0.3302
- net class Default: via_dia 0.6096 -> 0.6858; via_drill 0.3048 -> 0.3302
- board text added: "+"
- board text added: "GND"
- board text added: "ID"
- board text added: "USB+"
- board text added: "USB-"
- board text added: "VBUS"

Commit message: Switch matrix complete.
Parts:
- removed D50: D, Diodes_SMD:MiniMELF_Standard
- P4, R1, SW1: moved to B.Cu
- moved R1 208.4 mm to (183.5, 40.6), turned to 90 degrees
- moved SW1 192.4 mm to (191.0, 40.6), turned to 180 degrees
- moved P4 162.6 mm to (258.6, 42.9), turned to 270 degrees
- moved D32 7.49 mm to (311.8, 61.0)
- moved D10 0.94 mm to (254.6, 33.7)
Routing:
- net C14: track 0.00 -> 248.1 mm, vias 0 -> 3
- net C13: track 83.2 -> 226.5 mm, vias 0 -> 4
- net RESET: track 0.00 -> 121.9 mm, vias 0 -> 4
- net R1: track 252.4 -> 371.2 mm, vias 0 -> 5
- net C12: track 87.1 -> 199.7 mm, vias 0 -> 4
- net C11: track 87.0 -> 189.4 mm, vias 0 -> 5
- net R4: track 374.8 -> 415.8 mm, vias 2 -> 4
- net +5V: track 124.0 -> 164.7 mm, vias 0 -> 3
- net R3: track 341.8 -> 375.6 mm
- net AUDIO: track 0.00 -> 26.5 mm
- net Net-(D49-Pad2): track 3.16 -> 20.2 mm, vias 0 -> 1
- net Net-(D67-Pad2): track 3.16 -> 16.3 mm
- net Net-(D32-Pad2): track 0.00 -> 12.4 mm
- net Net-(D10-Pad2): track 0.00 -> 10.9 mm
- net GND: track 0.51 -> 2.23 mm, vias 0 -> 1
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Other:
- rule trace_min: 0.2032 -> 0.1905
